Commit message: Simple panda+drone rviz simulator

File: urdfs/panda_arm_hand.urdf (robot description, URDF)
Before this commit: robot panda, 14 links, 13 joints
Joints:
- removed joint panda_gripper
- added joint panda_gripper_joint: type fixed, parent panda_link8, child panda_gripper, origin xyz=-0.000 -0.000 0.103 rpy=3.1416 0.000 -0.785, axis 0 0 0
