Commit message: fixes for new point cloud and urdf

File: urdfs/panda.urdf (robot description, URDF)
Before this commit: robot panda_kinect, 16 links, 15 joints
Links:
- added link panda_gripper
Joints:
- added joint panda_gripper_joint: type fixed, parent panda_link8, child panda_gripper, origin xyz=-0.000 -0.000 0.103 rpy=3.1416 0.000 -0.785, axis 0 0 0
